File: Interface/Interface.kicad_sch (KiCad schematic)
At the start: 0 parts

Commit message: Add Symbols of FPGA and MCU
Parts:
- added C1, C16, C18, C2, C3, C4: 10u, Capacitor_SMD:C_0402_1005Metric, symbol Device:C
- added C10, C12, C14, C15, C20, C5, C8: 4.7u, Capacitor_SMD:C_0402_1005Metric, symbol Device:C
- added C11, C19, C21, C6, C7, C9: 100n, Capacitor_SMD:C_0402_1005Metric, symbol Device:C
- added C13: 1u, Capacitor_SMD:C_0402_1005Metric, symbol Device:C
- added C17: 15p, Capacitor_SMD:C_0402_1005Metric, symbol Device:C
- added D1: PRTR5V0U2X, Package_TO_SOT_SMD:SOT-143, symbol Power_Protection:PRTR5V0U2X
- added J1: USB_C_Receptacle_USB2.0_16P, Connector_USB:USB_C_Receptacle_GCT_USB4110, symbol Connector:USB_C_Receptacle_USB2.0_16P
- added L1, L2: 1u, Inductor_SMD:L_Murata_DFE201610P, symbol Device:L
- added R1, R2, R6: 100k, Resistor_SMD:R_0402_1005Metric, symbol Device:R
- added R3: 499k, Resistor_SMD:R_0402_1005Metric, symbol Device:R
- added R4, R7: 5.1k, Resistor_SMD:R_0402_1005Metric, symbol Device:R
- added R5: 453k, Resistor_SMD:R_0402_1005Metric, symbol Device:R
- added R8: 100, Resistor_SMD:R_0402_1005Metric, symbol Device:R
- added R9: 12k, Resistor_SMD:R_0402_1005Metric, symbol Device:R
- added U1: ICE40UP5K-SG48ITR, Package_DFN_QFN:QFN-48-1EP_7x7mm_P0.5mm_EP5.6x5.6mm, symbol FPGA_Lattice:ICE40UP5K-SG48ITR
- added U2: USB3300-EZK, Package_DFN_QFN:QFN-32-1EP_5x5mm_P0.5mm_EP3.45x3.45mm, symbol Interface_USB:USB3300-EZK
- added U4, U5: TPS62A01ADRL, Package_TO_SOT_SMD:SOT-563, symbol Regulator_Switching:TPS62A01ADRL
- added U6: W25Q16JVUX, Package_SON:Winbond_USON-8-1EP_3x2mm_P0.5mm_EP0.2x1.6mm, symbol Memory_Flash:W25Q16JVSS
- added Y1, Y2: SiT8008xx-1x-xxE, Oscillator:Oscillator_SMD_SiT_PQFN-4Pin_2.5x2.0mm, symbol Oscillator:SiT8008xx-1x-xxE
- added Y3: ASCO, Oscillator:Oscillator_SMD_Abracon_ASCO-4Pin_1.6x1.2mm, symbol Oscillator:ASCO
Connections:
- new net: U1.14 (IOB_32a_SPI_SO), U6.2 (DO/IO_{1})
- new net: U1.15 (IOB_34a_SPI_SCK), U6.6 (CLK)
- new net: U1.16 (IOB_35b_SPI_SS), U6.1 (~{CS})
- new net: U1.17 (IOB_33b_SPI_SI), U6.5 (DI/IO_{0})
- new net: R1.2, R2.1, U4.5 (FB)
- new net: L2.1, U5.2 (SW)
- new net: R5.2, R6.1, U5.5 (FB)
- new net: J1.A5 (CC1), R7.2
- new net: J1.B5 (CC2), R4.2
- new net: C14.2, U2.29 (VDDA1.8)
- new net: C15.1, U2.15 (VDD1.8), U2.26 (VDD1.8)
- new net: R8.2, U1.29 (VCCPLL), U1.30 (VCC), U1.5 (VCC)
- new net: L1.1, U4.2 (SW)
- new net: R9.1, U2.32 (RBIAS)
- new net +1V2: C2.1, L1.2, R1.1
- new net +3V3: C10.1, C11.2, C12.1, C13.1, C18.1, C19.2, C20.2, C21.2, C4.1, C5.1, C6.2, C7.2, C8.1, C9.2, L2.2, R5.1, R8.1, U1.1 (VCCIO_2), U1.22 (SPI_VCCIO1), U1.24 (VPP_2V5), U1.33 (VCCIO_0), U2.16 (VDD3.3), U2.25 (VDD3.3), U2.30 (VDD3.3), U2.31 (REG_EN), U2.6 (VDD3.3), U6.8 (VCC), Y3.1 (Tri-State), Y3.4 (VDD)
- new net 24M: C17.1, U2.28 (XI), Y3.3 (OUT)
- new net GND: C1.2, C10.2, C11.1, C12.2, C13.2, C14.1, C15.2, C16.1, C17.2, C18.2, C19.1, C2.2, C20.1, C3.2, C4.2, C5.2, C6.1, C7.1, C8.2, C9.1, D1.1 (GND), J1.A1 (GND), J1.A12 (GND), J1.B1 (GND), J1.B12 (GND), J1.S1 (SHIELD), R2.2, R4.1, R6.2, R7.1, R9.2, U1.49 (GND), U2.1 (GND), U2.2 (GND), U2.33 (GND), U4.1 (GND), U5.1 (GND), U6.4 (GND), Y3.2 (GND)
- new net PGOOD: R3.2, U4.6 (PG), U5.4 (EN)
- new net USB_DM: D1.3 (I/O2), J1.A7 (D-), J1.B7 (D-), U2.8 (DM)
- new net USB_DP: D1.2 (I/O1), J1.A6 (D+), J1.B6 (D+), U2.7 (DP)
- new net VBUS: C1.1, C16.2, C3.1, D1.4 (VCC), J1.A4 (VBUS), J1.A9 (VBUS), J1.B4 (VBUS), J1.B9 (VBUS), R3.1, U2.4 (VBUS), U4.3 (VIN), U4.4 (EN), U5.3 (VIN)
- no-connect marks 0 -> 9
